File: board/_autosave-board.kicad_pcb (KiCad board)
At the start: 2 copper layers, 66.1 x 100.8 mm, 27 parts, among them J1 port attiny, J10 BMS Bat +, J11 BMS Bat gnd, J12 BMS out -, J13 BMS in +5v, J14 BMS in gnd, J15_C189893 BMS led charge ok, J16 Mp3 D1 led marche ok, J17_C189893 Haut parleur, J18_C189893 Batterie + et -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

Commit message: pcb carte mere mise a jour
Parts:
- renumbered J17_C189893 to J17, J18_C189893 to J18, J19_C189893 to J19, J21_C189893 to J21, J5_C189893 to J5
Routing:
- net GND: track 135.5 -> 131.8 mm, vias 3 -> 2
- net Net-(J7-Pin_1): track 52.9 -> 54.0 mm
Changed lines of the file:
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@@
 		)
 		(property "Value" "step up in +"
-			(at 0 -2.51 90)
+			(at -3.32 -2.94 90)
 			(layer "F.SilkS")
 			(effects
@@
 		(descr "Through hole straight pin header, 1x02, 2.54mm pitch, single row")
 		(tags "Through hole pin header THT 1x02 2.54mm single row")
-		(property "Reference" "J5_C189893"
+		(property "Reference" "J5"
 			(at 0 -2.38 0)
 			(layer "F.SilkS")
@@
 		(descr "JST GH series connector, BM02B-GHS-TBT (http://www.jst-mfg.com/product/pdf/eng/eGH.pdf), generated with kicad-footprint-generator")
 		(tags "connector JST GH vertical")
-		(property "Reference" "J17_C189893"
+		(property "Reference" "J17"
 			(at 0 -4 180)
 			(layer "F.SilkS")
@@
 		)
 		(property "Value" "step up in -"
-			(at 3.14 4.52 180)
+			(at -3.86 3.02 270)
 			(layer "F.SilkS")
 			(effects
@@
 		(descr "JST GH series connector, BM02B-GHS-TBT (http://www.jst-mfg.com/product/pdf/eng/eGH.pdf), generated with kicad-footprint-generator")
 		(tags "connector JST GH vertical")
-		(property "Reference" "J18_C189893"
+		(property "Reference" "J18"
 			(at 0 -4 0)
 			(layer "F.SilkS")
@@
 		(descr "JST GH series connector, BM02B-GHS-TBT (http://www.jst-mfg.com/product/pdf/eng/eGH.pdf), generated with kicad-footprint-generator")
 		(tags "connector JST GH vertical")
-		(property "Reference" "J19_C189893"
+		(property "Reference" "J19"
 			(at 0 -4 0)
 			(layer "F.SilkS")
@@
 		(descr "JST GH series connector, BM02B-GHS-TBT (http://www.jst-mfg.com/product/pdf/eng/eGH.pdf), generated with kicad-footprint-generator")
 		(tags "connector JST GH vertical")
-		(property "Reference" "J21_C189893"
+		(property "Reference" "J21"
 			(at 0 -4 180)
 			(layer "F.SilkS")
@@
 	)
 	(segment
-		(start 111.48 96.52)
-		(end 111.5 96.5)
-		(width 0.5)
-		(layer "F.Cu")
-		(net 2)
-	)
-	(segment
 		(start 107.95 96.52)
 		(end 107.95 98.05)
@@
 	)
 	(segment
-		(start 107.95 96.52)
-		(end 111.48 96.52)
-		(width 0.5)
-		(layer "F.Cu")
-		(net 2)
-	)
-	(segment
 		(start 92 107.5)
 		(end 92.5 107)
@@
 	)
 	(via
-		(at 111.5 96.5)
+		(at 109.5 70)
 		(size 0.6)
 		(drill 0.3)
@@
 		(net 2)
 	)
-	(via
-		(at 109.5 70)
-		(size 0.6)
-		(drill 0.3)
-		(layers "F.Cu" "B.Cu")
+	(segment
+		(start 109.5 70)
+		(end 109.5 94.97)
+		(width 0.5)
+		(layer "B.Cu")
 		(net 2)
 	)
@@
 	)
 	(segment
-		(start 109.5 82.5)
-		(end 109.5 70)
-		(width 0.5)
-		(layer "B.Cu")
-		(net 2)
-	)
-	(segment
-		(start 111.5 96.5)
-		(end 111.5 84.5)
+		(start 109.5 94.97)
+		(end 107.95 96.52)
 		(width 0.5)
 		(layer "B.Cu")
@@
 	)
 	(segment
-		(start 111.5 84.5)
-		(end 109.5 82.5)
-		(width 0.5)
-		(layer "B.Cu")
-		(net 2)
-	)
-	(segment
 		(start 107.5 61.5)
 		(end 112.625 56.375)
@@
 	)
 	(segment
-		(start 92.271 41.051)
-		(end 90.97 39.75)
+		(start 100 79.5)
+		(end 100 69)
+		(width 0.5)
+		(layer "B.Cu")
+		(net 11)
+	)
+	(segment
+		(start 94.5 63.5)
+		(end 94.5 41.5)
 		(width 0.5)
 		(layer "B.Cu")
@@
 	)
 	(segment
-		(start 92.271 71.771)
-		(end 92.271 41.051)
+		(start 94.5 41.5)
+		(end 92.75 39.75)
 		(width 0.5)
 		(layer "B.Cu")
@@
 	(segment
 		(start 101.5 81)
-		(end 92.271 71.771)
+		(end 100 79.5)
+		(width 0.5)
+		(layer "B.Cu")
+		(net 11)
+	)
+	(segment
+		(start 92.75 39.75)
+		(end 90.97 39.75)
+		(width 0.5)
+		(layer "B.Cu")
+		(net 11)
+	)
+	(segment
+		(start 100 69)
+		(end 94.5 63.5)
 		(width 0.5)
 		(layer "B.Cu")
