File: board/board.kicad_pcb (KiCad board)
At the start: 2 copper layers, 58 x 75 mm, 29 parts, among them J1 port attiny, J10 BMS Bat +, J11 BMS Bat gnd, J12 BMS out -, J13 BMS in +5v, J14 BMS in gnd, J15 alim mp3 -, J16 SWDIO, J17 next, J18 vol -, J19 SWIM, J2 Conn_01x02_Pin, J24 port 3-C265421, J3 alim mp3 +, J4 hp mp3, J5 step out - gnd, J6 step up out+, J7 step up in +, J8 step up in -, J9 BMS out +, U1 ATtiny85-20S, U2 ATtiny85V-10P, U3 STM8S001J3M, U4 CH32V003AxMx

Commit message: passage du code CH32 a core officiel WCH Arduino https://github.com/openwch/board_manager_files/raw/main/package_ch32v_index.json
Routing:
- net GND: track 187.9 -> 197.3 mm, vias 16 -> 17
Changed lines of the file:
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@@
+	)
+	(segment
+		(start 76.4 80.9)
+		(end 76.4 80.88)
+		(width 0.5)
+		(layer "F.Cu")
+		(net 2)
 	)
 	(segment
@@
 	)
 	(segment
+		(start 76.4 80.88)
+		(end 74.5 78.98)
+		(width 0.5)
+		(layer "F.Cu")
+		(net 2)
+	)
+	(segment
 		(start 92.58 52.91)
 		(end 92.54 52.95)
@@
 	)
 	(segment
+		(start 77.955735 82.455735)
+		(end 76.4 80.9)
+		(width 0.5)
+		(layer "F.Cu")
+		(net 2)
+	)
+	(segment
 		(start 100.225 53.375)
 		(end 100.6 53)
@@
 	)
 	(via
+		(at 77.955735 82.455735)
+		(size 0.6)
+		(drill 0.3)
+		(layers "F.Cu" "B.Cu")
+		(net 2)
+	)
+	(via
 		(at 79.41 101.13)
 		(size 0.6)
@@
 	)
 	(segment
+		(start 79.955735 82.455735)
+		(end 81.73 84.23)
+		(width 0.5)
+		(layer "B.Cu")
+		(net 2)
+	)
+	(segment
 		(start 99.561 60.349)
 		(end 97.169 60.349)
@@
 		(width 0.5)
 		(layer "B.Cu")
+		(net 2)
+	)
+	(segment
+		(start 77.955735 82.455735)
+		(end 79.955735 82.455735)
+		(width 0.5)
+		(layer "B.Cu")
