File: board/board-backups/board-2026-06-30_212628/_autosave-board.kicad_sch (KiCad schematic)
At the start: 29 parts, among them J1 port attiny, J10 BMS Bat +, J11 BMS Bat gnd, J12 BMS out -, J13 BMS in +5v, J14 BMS in gnd, J15 alim mp3 -, J16 SWDIO, J17 next, J18 vol -, J19 SWDIO, J2 Conn_01x02_Pin, J24 port 3-C265421, J3 alim mp3 +, J4 hp mp3, J5 step out - gnd, J6 step up out+, J7 step up in +, J8 step up in -, J9 BMS out +, U1 ATtiny85-20S, U2 ATtiny85V-10P, U3 STM8S001J3M, U4 CH32V003AxMx

Commit message: bug pcb + broche de programmation
Parts:
- J19: value SWDIO -> SWIM
Changed lines of the file:
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@@
 			)
 		)
-		(property "Value" "SWDIO"
+		(property "Value" "SWIM"
 			(at 175.895 133.35 0)
 			(effects
