File: board/board-backups/board-2026-06-30_212628/board-backups/board-2026-06-11_233831-(1)/board.kicad_pcb (KiCad board)
At the start: 2 copper layers, 58 x 75 mm, 29 parts, among them J1 port attiny, J10 BMS Bat +, J11 BMS Bat gnd, J12 BMS out -, J13 BMS in +5v, J14 BMS in gnd, J15 alim mp3 -, J16 SWDIO, J17 next, J18 vol -, J19 SWIM, J2 Conn_01x02_Pin, J24 port 3-C265421, J3 alim mp3 +, J4 hp mp3, J5 step out - gnd, J6 step up out+, J7 step up in +, J8 step up in -, J9 BMS out +, U1 ATtiny85-20S, U2 ATtiny85V-10P, U3 STM8S001J3M, U4 CH32V003AxMx

Commit message: bug pcb + broche de programmation
Parts:
- removed J16: SWDIO, Connector_PinHeader_2.54mm:PinHeader_1x01_P2.54mm_Vertical
- removed J19: SWIM, Connector_PinHeader_2.54mm:PinHeader_1x01_P2.54mm_Vertical
- moved J15 5.40 mm to (79.9, 79.0)
- moved J3 5.40 mm to (74.5, 79.0)
Connections:
- U3 pad 8: Net-(J19-Pin_1) -> unconnected-(U3-PD5-Pad8)
- U4 pad 7: Net-(J16-Pin_1) -> unconnected-(U4-PD1-Pad7)
Routing:
- net GND: track 187.9 -> 154.2 mm, vias 16 -> 14
- net Net-(J19-Pin_1): track 22.2 -> 0.00 mm, vias 4 -> 0
- net Net-(J16-Pin_1): track 22.0 -> 0.00 mm, vias 2 -> 0
- net VCC: track 160.9 -> 175.5 mm, vias 6 -> 3
- net vol - mp3: track 148.6 -> 144.2 mm
Other:
- board size 58 x 75 mm -> 42.6 x 75.4 mm
- board text removed: "vcc"
