File: board/board-backups/board-2026-06-30_212628/board-backups/board-2026-06-11_233831-(1)/board.kicad_sch (KiCad schematic)
At the start: 29 parts, among them J1 port attiny, J10 BMS Bat +, J11 BMS Bat gnd, J12 BMS out -, J13 BMS in +5v, J14 BMS in gnd, J15 alim mp3 -, J16 SWDIO, J17 next, J18 vol -, J19 SWDIO, J2 Conn_01x02_Pin, J24 port 3-C265421, J3 alim mp3 +, J4 hp mp3, J5 step out - gnd, J6 step up out+, J7 step up in +, J8 step up in -, J9 BMS out +, U1 ATtiny85-20S, U2 ATtiny85V-10P, U3 STM8S001J3M, U4 CH32V003AxMx

Commit message: bug pcb + broche de programmation
Parts:
- removed J16, J19: SWDIO, Connector_PinHeader_2.54mm:PinHeader_1x01_P2.54mm_Vertical, symbol Connector:Conn_01x01_Pin
Changed lines of the file:
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@@
 	(wire
 		(pts
-			(xy 171.45 124.46) (xy 171.45 135.89)
-		)
-		(stroke
-			(width 0)
-			(type default)
-		)
-	)
-	(wire
-		(pts
 			(xy 242.57 151.13) (xy 261.62 151.13)
 		)
@@
 	(wire
 		(pts
-			(xy 167.64 124.46) (xy 171.45 124.46)
-		)
-		(stroke
-			(width 0)
-			(type default)
-		)
-	)
-	(wire
-		(pts
 			(xy 92.71 27.94) (xy 95.25 27.94)
 		)
@@
 	(wire
 		(pts
-			(xy 255.27 80.01) (xy 264.16 80.01)
-		)
-		(stroke
-			(width 0)
-			(type default)
-		)
-	)
-	(wire
-		(pts
 			(xy 80.01 86.36) (xy 105.41 86.36)
 		)
@@
 	(symbol
 		(lib_id "Connector:Conn_01x01_Pin")
-		(at 269.24 80.01 0)
-		(mirror y)
-		(unit 1)
-		(exclude_from_sim no)
-		(in_bom yes)
-		(on_board yes)
-		(dnp no)
-		(fields_autoplaced yes)
-		(property "Reference" "J16"
-			(at 268.605 74.93 0)
-			(effects
-				(font
-					(size 1.27 1.27)
-				)
-			)
-		)
-		(property "Value" "SWDIO"
-			(at 268.605 77.47 0)
-			(effects
-				(font
-					(size 1.27 1.27)
-				)
-			)
-		)
-		(property "Footprint" "Connector_PinHeader_2.54mm:PinHeader_1x01_P2.54mm_Vertical"
-			(at 269.24 80.01 0)
-			(effects
-				(font
-					(size 1.27 1.27)
-				)
-				(hide yes)
-			)
-		)
-		(property "Datasheet" "~"
-			(at 269.24 80.01 0)
-			(effects
-				(font
-					(size 1.27 1.27)
-				)
-				(hide yes)
-			)
-		)
-		(property "Description" "Generic connector, single row, 01x01, script generated"
-			(at 269.24 80.01 0)
-			(effects
-				(font
-					(size 1.27 1.27)
-				)
-				(hide yes)
-			)
-		)
-		(pin "1"
-		)
-		(instances
-			(project "board"
-				(path "/1d4ba15b-5ce7-48af-a486-6050b996f974"
-					(reference "J16")
-					(unit 1)
-				)
-			)
-		)
-	)
-	(symbol
-		(lib_id "Connector:Conn_01x01_Pin")
 		(at 53.34 91.44 0)
 		(mirror x)
@@
 					(unit 1)
 				)
-			)
-		)
-	)
-	(symbol
-		(lib_id "Connector:Conn_01x01_Pin")
-		(at 176.53 135.89 0)
-		(mirror y)
-		(unit 1)
-		(exclude_from_sim no)
-		(in_bom yes)
-		(on_board yes)
-		(dnp no)
-		(fields_autoplaced yes)
-		(property "Reference" "J19"
-			(at 175.895 130.81 0)
-			(effects
-				(font
-					(size 1.27 1.27)
-				)
-			)
-		)
-		(property "Value" "SWDIO"
-			(at 175.895 133.35 0)
-			(effects
-				(font
-					(size 1.27 1.27)
-				)
-			)
-		)
-		(property "Footprint" "Connector_PinHeader_2.54mm:PinHeader_1x01_P2.54mm_Vertical"
-			(at 176.53 135.89 0)
-			(effects
-				(font
-					(size 1.27 1.27)
-				)
-				(hide yes)
-			)
-		)
-		(property "Datasheet" "~"
-			(at 176.53 135.89 0)
-			(effects
-				(font
-					(size 1.27 1.27)
-				)
-				(hide yes)
-			)
-		)
-		(property "Description" "Generic connector, single row, 01x01, script generated"
-			(at 176.53 135.89 0)
-			(effects
-				(font
-					(size 1.27 1.27)
-				)
-				(hide yes)
-			)
-		)
-		(pin "1"
-		)
-		(instances
-			(project "board"
-				(path "/1d4ba15b-5ce7-48af-a486-6050b996f974"
-					(reference "J19")
-					(unit 1)
-				)
